File: KiCad/Centauri.kicad_pcb (KiCad board)
At the start: 2 copper layers, 299.2 x 90.4 mm, 147 parts, among them U1 Raspberry_Pi_Pico

Commit message: Add files via upload
Parts:
- removed D67: Diode, ScottoKeebs_Components:Diode_SOD-123
- removed VR1, VR2: RK1191124001, RK1191124001:RK1191124001
- added U2: 482020514001, 482020514001:482020514001, F.Cu at (273.4, 46.1)
- moved D66 14.8 mm to (270.2, 50.1)
- moved D12 4.30 mm to (263.5, 44.5)
Connections:
- D66 pad 2: Row 2 -> Row 1
- U1 pad 32: Potentiometer 1 -> Signal A
- U1 pad 34: Potentiometer 2 -> Signal B
Routing:
- net Potentiometer 1: track 56.5 -> 0.00 mm, vias 1 -> 0
- net Signal B: track 0.00 -> 51.2 mm, vias 0 -> 1
- net Potentiometer 2: track 48.4 -> 0.00 mm, vias 1 -> 0
- net GND: track 105.6 -> 58.2 mm, vias 5 -> 6
- net 3.3V: track 98.9 -> 52.4 mm
- net Signal A: track 0.00 -> 40.5 mm, vias 0 -> 1
- net Net-(D67-K): track 16.3 -> 0.00 mm, vias 1 -> 0
- net Column 13: track 181.1 -> 193.7 mm
- net Row 1: track 326.5 -> 322.3 mm
- net Net-(D12-K): track 23.2 -> 27.2 mm
- net Row 2: track 339.6 -> 336.7 mm
- net Net-(D66-K): track 8.65 -> 6.12 mm
